File: MinimalDuino.brd (EAGLE design)
At the start: 25 x 35 mm, 16 parts, among them J1 AVR_SPI_PRG_6PTH, U1 ATMEGA328P

Commit message: Board and schematic updates
Board and schematic updates
Parts:
- S1: value SWITCH-MOMENTARY-2SIDE_EZ -> SW
Connections:
- net MISO renamed D12/MISO
- net MOSI renamed D11/MOSI
- net SCK renamed D13/SCK
Changed lines of the file:
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@@
 <element name="Y1" library="SparkFun-FreqCtrl" package="HC49US" value="" x="12.7" y="24.368125"/>
 <element name="J1" library="SparkFun-Connectors" package="2X3" value="AVR_SPI_PRG_6PTH" x="12.065" y="2"/>
-<element name="S1" library="SparkFun-Electromechanical" package="TACTILE-PTH-SIDEEZ" value="SWITCH-MOMENTARY-2SIDE_EZ" x="5.5" y="32.9825" rot="R180"/>
+<element name="S1" library="SparkFun-Electromechanical" package="TACTILE-PTH-SIDEEZ" value="SW" x="5.5" y="32.9825" rot="R180"/>
 <element name="R2" library="SparkFun-Passives" package="0805" value="" x="8.7" y="5" rot="R180"/>
 <element name="R3" library="SparkFun-Passives" package="0805" value="" x="13.25" y="31.4" rot="R180"/>
@@
 <contactref element="JP2" pad="9"/>
 <wire x1="16.9926" y1="16.77" x2="16.9926" y2="18.2626" width="0.2" layer="1"/>
-<wire x1="16.9926" y1="18.2626" x2="17.62125" y2="18.89125" width="0.2" layer="1"/>
-<via x="17.62125" y="18.89125" extent="1-16" drill="0.31"/>
-<wire x1="17.62125" y1="18.89125" x2="19.27125" y2="18.89125" width="0.2" layer="16"/>
-<wire x1="19.27125" y1="18.89125" x2="19.77125" y2="18.89125" width="0.2" layer="16"/>
+<via x="19.288125" y="18.89125" extent="1-16" drill="0.31"/>
+<wire x1="19.288125" y1="18.89125" x2="19.27125" y2="18.89125" width="0.2" layer="16"/>
+<wire x1="19.27125" y1="18.89125" x2="19.288125" y2="18.89125" width="0.2" layer="16"/>
+<wire x1="19.288125" y1="18.89125" x2="19.77125" y2="18.89125" width="0.2" layer="16"/>
 <wire x1="19.77125" y1="18.89125" x2="23.2" y2="22.32" width="0.2" layer="16"/>
+<wire x1="19.288125" y1="18.89125" x2="17.62125" y2="18.89125" width="0.2" layer="1"/>
+<wire x1="17.62125" y1="18.89125" x2="16.9926" y2="18.2626" width="0.2" layer="1"/>
 </signal>
 <signal name="D3">
@@
 <via x="16.66875" y="19.3675" extent="1-16" drill="0.31"/>
 <wire x1="16.66875" y1="19.3675" x2="17.145" y2="19.84375" width="0.2" layer="16"/>
-<wire x1="17.145" y1="19.84375" x2="19.05" y2="19.84375" width="0.2" layer="16"/>
-<wire x1="19.05" y1="19.84375" x2="19.446875" y2="20.240625" width="0.2" layer="16"/>
-<wire x1="19.446875" y1="20.240625" x2="19.446875" y2="23.574375" width="0.2" layer="16"/>
+<wire x1="17.145" y1="19.84375" x2="18.7325" y2="19.84375" width="0.2" layer="16"/>
+<wire x1="18.7325" y1="19.84375" x2="19.446875" y2="20.558125" width="0.2" layer="16"/>
+<wire x1="19.446875" y1="20.558125" x2="19.446875" y2="23.574375" width="0.2" layer="16"/>
 <wire x1="19.446875" y1="23.574375" x2="20.7325" y2="24.86" width="0.2" layer="16"/>
 <wire x1="20.7325" y1="24.86" x2="23.2" y2="24.86" width="0.2" layer="16"/>
@@
 <wire x1="2.15875" y1="9.62" x2="2.65875" y2="10.12" width="0.2" layer="1"/>
 </signal>
-<signal name="SCK">
+<signal name="D13/SCK">
 <contactref element="J1" pad="3"/>
 <contactref element="U1" pad="17"/>
@@
 <wire x1="10.00125" y1="1.349375" x2="6.746875" y2="1.349375" width="0.2" layer="1"/>
 </signal>
-<signal name="MISO">
+<signal name="D12/MISO">
 <contactref element="J1" pad="1"/>
 <contactref element="U1" pad="16"/>
@@
 <wire x1="15.64" y1="14.37" x2="16.9926" y2="14.37" width="0" layer="19" extent="1-1"/>
 </signal>
-<signal name="MOSI">
+<signal name="D11/MOSI">
 <contactref element="J1" pad="4"/>
 <contactref element="U1" pad="15"/>
@@
 <wire x1="14.605" y1="4.54" x2="14.605" y2="5.715" width="0.2" layer="16"/>
 <wire x1="14.605" y1="5.715" x2="12.7" y2="7.62" width="0.2" layer="16"/>
-<wire x1="12.7" y1="7.62" x2="1.84" y2="7.62" width="0.2" layer="16"/>
+<wire x1="12.7" y1="7.62" x2="2.31625" y2="7.62" width="0.2" layer="16"/>
 <contactref element="JP3" pad="3"/>
 <wire x1="3.4925" y1="9.2725" x2="3.4925" y2="9.128125" width="0.2" layer="1"/>
@@
 <wire x1="1.984375" y1="7.62" x2="1.984375" y2="7.264375" width="0.2" layer="1"/>
 <wire x1="1.984375" y1="7.264375" x2="1.8" y2="7.08" width="0.2" layer="1"/>
-<wire x1="1.84" y1="7.62" x2="1.84" y2="7.12" width="0.2" layer="16"/>
+<wire x1="2.31625" y1="7.62" x2="1.84" y2="7.12" width="0.2" layer="16"/>
 <wire x1="1.84" y1="7.12" x2="1.8" y2="7.08" width="0.2" layer="16"/>
 </signal>
